File: CPX-Breakout/CPX-Breakout.sch (KiCad schematic (older format))
At the start: 14 parts, among them J1 3.3V, J10 A6_Rx, J11 3.3V, J12 A5_SDA, J13 A4_SCL, J14 GND, J2 A3, J3 A2, J4 GND, J5 A1, J6 A0, J7 Vout, J8 GND, J9 A7_Tx

Commit message: Deactivated contact pads for SPICE
Deactivated the contacts for SPICE simulation so that the existing connectors do not interfere with the simulator.
Parts:
- J1, J11: Spice_Model (none) -> 3.3V; Spice_Netlist_Enabled (none) -> N; Spice_Primitive (none) -> J
- J10: Spice_Model (none) -> A6_Rx; Spice_Netlist_Enabled (none) -> N; Spice_Primitive (none) -> J
- J12: Spice_Model (none) -> A5_SDA; Spice_Netlist_Enabled (none) -> N; Spice_Primitive (none) -> J
- J13: Spice_Model (none) -> A4_SCL; Spice_Netlist_Enabled (none) -> N; Spice_Primitive (none) -> J
- J14, J4, J8: Spice_Model (none) -> GND; Spice_Netlist_Enabled (none) -> N; Spice_Primitive (none) -> J
- J2: Spice_Model (none) -> A3; Spice_Netlist_Enabled (none) -> N; Spice_Primitive (none) -> J
- J3: Spice_Model (none) -> A2; Spice_Netlist_Enabled (none) -> N; Spice_Primitive (none) -> J
- J5: Spice_Model (none) -> A1; Spice_Netlist_Enabled (none) -> N; Spice_Primitive (none) -> J
- J6: Spice_Model (none) -> A0; Spice_Netlist_Enabled (none) -> N; Spice_Primitive (none) -> J
- J7: Spice_Model (none) -> Vout; Spice_Netlist_Enabled (none) -> N; Spice_Primitive (none) -> J
- J9: Spice_Model (none) -> A7_Tx; Spice_Netlist_Enabled (none) -> N; Spice_Primitive (none) -> J
Changed lines of the file:
@@
 F 2 "CPX-Adapter:CPX-Pad" H 9150 1800 50  0001 C CNN
 F 3 "~" H 9150 1800 50  0001 C CNN
+F 4 "J" H 9150 1800 50  0001 C CNN "Spice_Primitive"
+F 5 "3.3V" H 9150 1800 50  0001 C CNN "Spice_Model"
+F 6 "N" H 9150 1800 50  0001 C CNN "Spice_Netlist_Enabled"
 	1    9150 1800
 	1    0    0    -1
@@
 F 2 "CPX-Adapter:CPX-Pad" H 9150 2050 50  0001 C CNN
 F 3 "~" H 9150 2050 50  0001 C CNN
+F 4 "J" H 9150 2050 50  0001 C CNN "Spice_Primitive"
+F 5 "A3" H 9150 2050 50  0001 C CNN "Spice_Model"
+F 6 "N" H 9150 2050 50  0001 C CNN "Spice_Netlist_Enabled"
 	1    9150 2050
 	1    0    0    -1
@@
 F 2 "CPX-Adapter:CPX-Pad" H 9150 2300 50  0001 C CNN
 F 3 "~" H 9150 2300 50  0001 C CNN
+F 4 "J" H 9150 2300 50  0001 C CNN "Spice_Primitive"
+F 5 "A2" H 9150 2300 50  0001 C CNN "Spice_Model"
+F 6 "N" H 9150 2300 50  0001 C CNN "Spice_Netlist_Enabled"
 	1    9150 2300
 	1    0    0    -1
@@
 F 2 "CPX-Adapter:CPX-Pad" H 9150 2550 50  0001 C CNN
 F 3 "~" H 9150 2550 50  0001 C CNN
+F 4 "J" H 9150 2550 50  0001 C CNN "Spice_Primitive"
+F 5 "GND" H 9150 2550 50  0001 C CNN "Spice_Model"
+F 6 "N" H 9150 2550 50  0001 C CNN "Spice_Netlist_Enabled"
 	1    9150 2550
 	1    0    0    -1
@@
 F 2 "CPX-Adapter:CPX-Pad" H 9150 2800 50  0001 C CNN
 F 3 "~" H 9150 2800 50  0001 C CNN
+F 4 "J" H 9150 2800 50  0001 C CNN "Spice_Primitive"
+F 5 "A1" H 9150 2800 50  0001 C CNN "Spice_Model"
+F 6 "N" H 9150 2800 50  0001 C CNN "Spice_Netlist_Enabled"
 	1    9150 2800
 	1    0    0    -1
@@
 F 2 "CPX-Adapter:CPX-Pad" H 9150 3050 50  0001 C CNN
 F 3 "~" H 9150 3050 50  0001 C CNN
+F 4 "J" H 9150 3050 50  0001 C CNN "Spice_Primitive"
+F 5 "A0" H 9150 3050 50  0001 C CNN "Spice_Model"
+F 6 "N" H 9150 3050 50  0001 C CNN "Spice_Netlist_Enabled"
 	1    9150 3050
 	1    0    0    -1
@@
 F 2 "CPX-Adapter:CPX-Pad" H 9150 3300 50  0001 C CNN
 F 3 "~" H 9150 3300 50  0001 C CNN
+F 4 "J" H 9150 3300 50  0001 C CNN "Spice_Primitive"
+F 5 "Vout" H 9150 3300 50  0001 C CNN "Spice_Model"
+F 6 "N" H 9150 3300 50  0001 C CNN "Spice_Netlist_Enabled"
 	1    9150 3300
 	1    0    0    -1
@@
 F 2 "CPX-Adapter:CPX-Pad" H 9150 3550 50  0001 C CNN
 F 3 "~" H 9150 3550 50  0001 C CNN
+F 4 "J" H 9150 3550 50  0001 C CNN "Spice_Primitive"
+F 5 "GND" H 9150 3550 50  0001 C CNN "Spice_Model"
+F 6 "N" H 9150 3550 50  0001 C CNN "Spice_Netlist_Enabled"
 	1    9150 3550
 	1    0    0    -1
@@
 F 2 "CPX-Adapter:CPX-Pad" H 9150 3800 50  0001 C CNN
 F 3 "~" H 9150 3800 50  0001 C CNN
+F 4 "J" H 9150 3800 50  0001 C CNN "Spice_Primitive"
+F 5 "A7_Tx" H 9150 3800 50  0001 C CNN "Spice_Model"
+F 6 "N" H 9150 3800 50  0001 C CNN "Spice_Netlist_Enabled"
 	1    9150 3800
 	1    0    0    -1
@@
 F 2 "CPX-Adapter:CPX-Pad" H 9150 4050 50  0001 C CNN
 F 3 "~" H 9150 4050 50  0001 C CNN
+F 4 "J" H 9150 4050 50  0001 C CNN "Spice_Primitive"
+F 5 "A6_Rx" H 9150 4050 50  0001 C CNN "Spice_Model"
+F 6 "N" H 9150 4050 50  0001 C CNN "Spice_Netlist_Enabled"
 	1    9150 4050
 	1    0    0    -1
@@
 F 2 "CPX-Adapter:CPX-Pad" H 9150 4300 50  0001 C CNN
 F 3 "~" H 9150 4300 50  0001 C CNN
+F 4 "J" H 9150 4300 50  0001 C CNN "Spice_Primitive"
+F 5 "3.3V" H 9150 4300 50  0001 C CNN "Spice_Model"
+F 6 "N" H 9150 4300 50  0001 C CNN "Spice_Netlist_Enabled"
 	1    9150 4300
 	1    0    0    -1
@@
 F 2 "CPX-Adapter:CPX-Pad" H 9150 4550 50  0001 C CNN
 F 3 "~" H 9150 4550 50  0001 C CNN
+F 4 "J" H 9150 4550 50  0001 C CNN "Spice_Primitive"
+F 5 "A5_SDA" H 9150 4550 50  0001 C CNN "Spice_Model"
+F 6 "N" H 9150 4550 50  0001 C CNN "Spice_Netlist_Enabled"
 	1    9150 4550
 	1    0    0    -1
@@
 F 2 "CPX-Adapter:CPX-Pad" H 9150 4800 50  0001 C CNN
 F 3 "~" H 9150 4800 50  0001 C CNN
+F 4 "J" H 9150 4800 50  0001 C CNN "Spice_Primitive"
+F 5 "A4_SCL" H 9150 4800 50  0001 C CNN "Spice_Model"
+F 6 "N" H 9150 4800 50  0001 C CNN "Spice_Netlist_Enabled"
 	1    9150 4800
 	1    0    0    -1
@@
 F 2 "CPX-Adapter:CPX-Pad" H 9150 5050 50  0001 C CNN
 F 3 "~" H 9150 5050 50  0001 C CNN
+F 4 "J" H 9150 5050 50  0001 C CNN "Spice_Primitive"
+F 5 "GND" H 9150 5050 50  0001 C CNN "Spice_Model"
+F 6 "N" H 9150 5050 50  0001 C CNN "Spice_Netlist_Enabled"
 	1    9150 5050
 	1    0    0    -1
